File: crimson.kicad_pcb (KiCad board)
At the start: 4 copper layers, 184 parts, among them J1 Conn_01x02_Socket, SW1 SW_Esc, SW10 SW_´, SW11 SW_1, SW12 SW_2, SW13 SW_3, SW14 SW_4, SW15 SW_5, SW16 SW_6, SW17 SW_7, SW18 SW_8, SW19 SW_F9, SW2 SW_F1, SW20 SW_F10, SW21 SW_Tab, SW22 SW_Capslock, SW23 SW_Q, SW24 SW_A, SW25 SW_W, SW26 SW_S, SW27 SW_E, SW28 SW_D, SW29 SW_R, SW3 SW_F2, SW30 SW_F, SW31 SW_T, SW32 SW_G, SW33 SW_Y, SW34 SW_H, SW35 SW_U, SW36 SW_J, SW37 SW_I, SW38 SW_K, SW39 SW_F11, SW4 SW_F3, SW40 SW_F12, SW41 SW_LShift, SW42 SW_LCtrl, SW43 SW_Insert, SW44 SW_Delete, SW45 SW_Z, SW46 SW_LMod, SW47 SW_Home, SW48 SW_End, SW49 SW_X, SW5 SW_F4, SW50 SW_LAlt, SW51 SW_PgUp, SW52 SW_PgDn, SW53 SW_C, SW54 SW_Space, SW55 SW_;, SW56 SW_-, SW57 SW_V, SW58 SW_RAlt, SW59 SW_', SW6 SW_F5, SW60 SW_+, SW61 SW_B, SW62 SW_RWin, SW63 SW_., SW64 SW_[, SW65 SW_N, SW66 SW_Push_Shielded, SW67 SW_/, SW68 SW_], SW69 SW_M, SW7 SW_F6, SW70 SW_RCtrl, SW71 SW_RShift, SW72 SW_\, SW73 SW_,, SW74 SW_L, SW75 SW_Backspace, SW76 SW_Enter, SW77 SW_PrtSc, SW78 SW_ScrollLock, SW79 SW_Pause, SW8 SW_F7, SW80 SW_9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

Commit message: [pcb] basic shape, diodes placement
Basic shape has been added to Edge.cuts, and
the diodes have been placed. Though I will probably put
the footprints on the back of the PCB in the future,
as to prevent possible collisions with the keycaps

Signed-off-by: Lucy Mielke <user@domain.tld>
Parts:
- SW92: moved to B.Cu
- moved D51 571.2 mm to (398.9, 105.9), turned to 90 degrees
- moved D52 569.1 mm to (399.1, 127.3), turned to 90 degrees
- moved D79 553.3 mm to (398.9, 74.1), turned to 90 degrees
- moved D47 548.6 mm to (377.8, 105.9), turned to 90 degrees
- moved D84 548.5 mm to (399.2, 191.0), turned to 90 degrees
- moved D85 547.9 mm to (399.0, 169.7), turned to 90 degrees
- moved D48 546.6 mm to (377.9, 127.3), turned to 90 degrees
- moved D78 545.4 mm to (377.8, 74.1), turned to 90 degrees
- moved D83 527.4 mm to (377.9, 191.0), turned to 90 degrees
- moved D81 526.9 mm to (377.9, 169.7), turned to 90 degrees
- moved D43 525.9 mm to (356.6, 105.9), turned to 90 degrees
- moved D44 524.1 mm to (356.4, 127.3), turned to 90 degrees
- moved D77 524.0 mm to (356.6, 74.1), turned to 90 degrees
- moved D82 506.4 mm to (356.7, 191.0), turned to 90 degrees
- moved D87 505.7 mm to (356.7, 169.6), turned to 90 degrees
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Other:
- board outline added: 388.9 x 165.2 mm

Commit message: [pcb] Add nice!nano stl, improve edge, move D* to back
Following changes were made:
- The nice!nano v2 footprint has a 3D model now
- The edge cuts were refined
- Diodes were moved to the back side of the board.

Signed-off-by: Lucy Mielke <user@domain.tld>
Parts:
- D1, D10, D11, D12, D13, D14, D15, D16, D17, D18, D19, D2, D20, D21, D22, D23, D24, D25, D26, D27, D28, D29, D3, D30, D31, D32, D33, D34, D35, D36, D37, D38, D39, D4, D40, D41, D42, D43, D44, D45, D46, D47, D48, D49, D5, D50, D51, D52, D53, D54, D55, D56, D57, D58, D59, D6, D60, D61, D62, D63, D64, D65, D66, D67, D68, D69, D7, D70, D71, D72, D73, D74, D75, D76, D77, D78, D79, D8, D80, D81, D82, D83, D84, D85, D86, D87, D88, D89, D9, D90: moved to B.Cu
- moved D54 6.10 mm to (175.8, 191.1), turned to 90 degrees
- moved J1 1.00 mm to (350.8, 42.3)
- moved SW91 1.00 mm to (363.3, 51.3)
- moved SW92 1.00 mm to (360.3, 36.2)
- moved U1 1.00 mm to (383.3, 43.9)
Other:
- outline, holes or cut-outs redrawn
