File: crimson.kicad_pcb (KiCad board)
At the start: 4 copper layers, 388.9 x 165.2 mm, 184 parts, among them J1 Conn_01x02_Socket, SW1 SW_Esc, SW10 SW_´, SW11 SW_1, SW12 SW_2, SW13 SW_3, SW14 SW_4, SW15 SW_5, SW16 SW_6, SW17 SW_7, SW18 SW_8, SW19 SW_F9, SW2 SW_F1, SW20 SW_F10, SW21 SW_Tab, SW22 SW_Capslock, SW23 SW_Q, SW24 SW_A, SW25 SW_W, SW26 SW_S, SW27 SW_E, SW28 SW_D, SW29 SW_R, SW3 SW_F2, SW30 SW_F, SW31 SW_T, SW32 SW_G, SW33 SW_Y, SW34 SW_H, SW35 SW_U, SW36 SW_J, SW37 SW_I, SW38 SW_K, SW39 SW_F11, SW4 SW_F3, SW40 SW_F12, SW41 SW_LShift, SW42 SW_LCtrl, SW43 SW_Insert, SW44 SW_Delete, SW45 SW_Z, SW46 SW_LMod, SW47 SW_Home, SW48 SW_End, SW49 SW_X, SW5 SW_F4, SW50 SW_LAlt, SW51 SW_PgUp, SW52 SW_PgDn, SW53 SW_C, SW54 SW_Space, SW55 SW_;, SW56 SW_-, SW57 SW_V, SW58 SW_RAlt, SW59 SW_', SW6 SW_F5, SW60 SW_+, SW61 SW_B, SW62 SW_RWin, SW63 SW_., SW64 SW_[, SW65 SW_N, SW66 SW_Push_Shielded, SW67 SW_/, SW68 SW_], SW69 SW_M, SW7 SW_F6, SW70 SW_RCtrl, SW71 SW_RShift, SW72 SW_\, SW73 SW_,, SW74 SW_L, SW75 SW_Backspace, SW76 SW_Enter, SW77 SW_PrtSc, SW78 SW_ScrollLock, SW79 SW_Pause, SW8 SW_F7, SW80 SW_9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

Commit message: [pcb] provisional routing
I routed everything, so I can see more easily how many pins I'd need
in order to split that thang in thirds for foldability

Signed-off-by: Lucy Mielke <user@domain.tld>
Parts:
- moved SW92 0.43 mm to (360.3, 36.6)
Routing:
- net ROW8: track 0.00 -> 639.9 mm, vias 0 -> 19
- net COL3: track 0.00 -> 631.4 mm, vias 0 -> 34
- net COL2: track 0.00 -> 603.6 mm, vias 0 -> 16
- net COL1: track 0.00 -> 600.0 mm, vias 0 -> 17
- net COL0: track 0.00 -> 588.1 mm, vias 0 -> 7
- net COL5: track 0.00 -> 571.0 mm, vias 0 -> 29
- net COL4: track 0.00 -> 568.7 mm, vias 0 -> 13
- net ROW5: track 0.00 -> 547.5 mm, vias 0 -> 11
- net COL6: track 0.00 -> 511.4 mm, vias 0 -> 16
- net ROW4: track 0.00 -> 497.6 mm, vias 0 -> 18
- net COL7: track 0.00 -> 486.7 mm, vias 0 -> 29
- net ROW1: track 0.00 -> 451.1 mm, vias 0 -> 12
- net ROW3: track 0.00 -> 450.5 mm, vias 0 -> 18
- net ROW2: track 0.00 -> 442.3 mm, vias 0 -> 18
- net ROW0: track 0.00 -> 425.7 mm, vias 0 -> 12
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- added copper zone on B.Cu, net GND
- added copper zone on F.Cu, net GND
- added copper zone on In1.Cu, net GND
- added copper zone on In2.Cu, net GND
