File: crimson.kicad_pcb (KiCad board)
At the start: 4 copper layers, 388.9 x 165.2 mm, 184 parts, among them J1 Conn_01x02_Socket, SW1 SW_Esc, SW10 SW_´, SW11 SW_1, SW12 SW_2, SW13 SW_3, SW14 SW_4, SW15 SW_5, SW16 SW_6, SW17 SW_7, SW18 SW_8, SW19 SW_F9, SW2 SW_F1, SW20 SW_F10, SW21 SW_Tab, SW22 SW_Capslock, SW23 SW_Q, SW24 SW_A, SW25 SW_W, SW26 SW_S, SW27 SW_E, SW28 SW_D, SW29 SW_R, SW3 SW_F2, SW30 SW_F, SW31 SW_T, SW32 SW_G, SW33 SW_Y, SW34 SW_H, SW35 SW_U, SW36 SW_J, SW37 SW_I, SW38 SW_K, SW39 SW_F11, SW4 SW_F3, SW40 SW_F12, SW41 SW_LShift, SW42 SW_LCtrl, SW43 SW_Insert, SW44 SW_Delete, SW45 SW_Z, SW46 SW_LMod, SW47 SW_Home, SW48 SW_End, SW49 SW_X, SW5 SW_F4, SW50 SW_LAlt, SW51 SW_PgUp, SW52 SW_PgDn, SW53 SW_C, SW54 SW_Space, SW55 SW_;, SW56 SW_-, SW57 SW_V, SW58 SW_RAlt, SW59 SW_', SW6 SW_F5, SW60 SW_+, SW61 SW_B, SW62 SW_RWin, SW63 SW_., SW64 SW_[, SW65 SW_N, SW66 SW_Push_Shielded, SW67 SW_/, SW68 SW_], SW69 SW_M, SW7 SW_F6, SW70 SW_RCtrl, SW71 SW_RShift, SW72 SW_\, SW73 SW_,, SW74 SW_L, SW75 SW_Backspace, SW76 SW_Enter, SW77 SW_PrtSc, SW78 SW_ScrollLock, SW79 SW_Pause, SW8 SW_F7, SW80 SW_9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

Commit message: [misc] add graphics and instructions for future non-exhausted me
I am tired, have a headache, and can't think straight. This is left for
future me to take care of

REMINDER: U still need mounting holes bruh

Signed-off-by: Lucy Mielke <user@domain.tld>
Routing:
- net ROW8: track 639.9 -> 0.00 mm, vias 19 -> 0
- net COL3: track 631.4 -> 0.00 mm, vias 34 -> 0
- net COL2: track 603.6 -> 0.00 mm, vias 16 -> 0
- net COL1: track 600.0 -> 0.00 mm, vias 17 -> 0
- net COL0: track 588.1 -> 0.00 mm, vias 7 -> 0
- net COL5: track 571.0 -> 0.00 mm, vias 29 -> 0
- net COL4: track 568.7 -> 0.00 mm, vias 13 -> 0
- net ROW5: track 547.5 -> 0.00 mm, vias 11 -> 0
- net COL6: track 511.4 -> 0.00 mm, vias 16 -> 0
- net ROW4: track 497.6 -> 0.00 mm, vias 18 -> 0
- net COL7: track 486.7 -> 0.00 mm, vias 29 -> 0
- net ROW1: track 451.1 -> 0.00 mm, vias 12 -> 0
- net ROW3: track 450.5 -> 0.00 mm, vias 18 -> 0
- net ROW2: track 442.3 -> 0.00 mm, vias 18 -> 0
- net ROW0: track 425.7 -> 0.00 mm, vias 12 -> 0
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Other:
- board text added: "${TITLE} ${REVISION} ${AUTHOR} licensed under ${LICENSE} ${COMMENT1}"
